File: OpticalTheremin.kicad_sch (KiCad schematic)
At the start: 6 parts, among them U1 VL6180X, U2 Lilygo_T7-S3, U3 MAX98357A

Commit message: finished routing, code draft 1 complete
Parts:
- RV1, RV2, RV3: footprint (none) -> Potentiometer_THT:Potentiometer_Bourns_PTA1543_Single_Slide
- U2: footprint (none) -> Module:LilyGo_T7-S3
- U3: footprint (none) -> Audio_Module:MAX98357A
Connections:
- net 3V3: now also U3.7 (Vin); no longer U3. (Vin)
- net BCLK: now also U3.2 (BCLK); no longer U3. (Vin)
- net DOUT: now also U3.3 (DIN); no longer U3. (Vin)
- net GND2: now also U3.6 (GND); no longer U3. (Vin)
- net LRC: now also U3.1 (LRC); no longer U3. (Vin)
- net SENSITIVITY: now also U2.16 (A2CH5); no longer U2.47
- net VIBRATO: now also U2.08 (A1CH7); no longer U2.46
- net VOLUME: now also U2.05 (A1CH4); no longer U2.45
Changed lines of the file:
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@@
+    (stroke (width 0) (type default) (color 0 0 0 0))
+  )
+  (wire (pts (xy 78.74 77.47) (xy 88.9 77.47))
     (stroke (width 0) (type default) (color 0 0 0 0))
   )
@@
     (stroke (width 0) (type default) (color 0 0 0 0))
   )
-  (wire (pts (xy 78.74 113.03) (xy 88.9 113.03))
+  (wire (pts (xy 78.74 62.23) (xy 88.9 62.23))
     (stroke (width 0) (type default) (color 0 0 0 0))
   )
@@
     (stroke (width 0) (type default) (color 0 0 0 0))
   )
+  (wire (pts (xy 48.26 130.81) (xy 48.26 137.16))
+    (stroke (width 0) (type default) (color 0 0 0 0))
+  )
+  (wire (pts (xy 62.23 57.15) (xy 62.23 76.2))
+    (stroke (width 0) (type default) (color 0 0 0 0))
+  )
+  (wire (pts (xy 49.53 97.79) (xy 49.53 104.14))
+    (stroke (width 0) (type default) (color 0 0 0 0))
+  )
+  (wire (pts (xy 31.75 83.82) (xy 45.72 83.82))
+    (stroke (width 0) (type default) (color 0 0 0 0))
+  )
+  (wire (pts (xy 45.72 57.15) (xy 62.23 57.15))
+    (stroke (width 0) (type default) (color 0 0 0 0))
+  )
+  (wire (pts (xy 78.74 73.66) (xy 88.9 73.66))
+    (stroke (width 0) (type default) (color 0 0 0 0))
+  )
+  (wire (pts (xy 31.75 64.77) (xy 31.75 83.82))
+    (stroke (width 0) (type default) (color 0 0 0 0))
+  )
+  (wire (pts (xy 45.72 130.81) (xy 45.72 137.16))
+    (stroke (width 0) (type default) (color 0 0 0 0))
+  )
+  (wire (pts (xy 45.72 64.77) (xy 31.75 64.77))
+    (stroke (width 0) (type default) (color 0 0 0 0))
+  )
+  (wire (pts (xy 133.35 81.28) (xy 140.97 81.28))
+    (stroke (width 0) (type default) (color 0 0 0 0))
+  )
+  (wire (pts (xy 31.75 101.6) (xy 45.72 101.6))
+    (stroke (width 0) (type default) (color 0 0 0 0))
+  )
+  (wire (pts (xy 31.75 83.82) (xy 31.75 101.6))
+    (stroke (width 0) (type default) (color 0 0 0 0))
+  )
   (wire (pts (xy 81.28 69.85) (xy 88.9 69.85))
     (stroke (width 0) (type default) (color 0 0 0 0))
   )
-  (wire (pts (xy 48.26 130.81) (xy 48.26 137.16))
-    (stroke (width 0) (type default) (color 0 0 0 0))
-  )
-  (wire (pts (xy 62.23 57.15) (xy 62.23 76.2))
-    (stroke (width 0) (type default) (color 0 0 0 0))
-  )
-  (wire (pts (xy 49.53 97.79) (xy 49.53 104.14))
-    (stroke (width 0) (type default) (color 0 0 0 0))
-  )
-  (wire (pts (xy 31.75 83.82) (xy 45.72 83.82))
-    (stroke (width 0) (type default) (color 0 0 0 0))
-  )
-  (wire (pts (xy 45.72 57.15) (xy 62.23 57.15))
-    (stroke (width 0) (type default) (color 0 0 0 0))
-  )
-  (wire (pts (xy 78.74 109.22) (xy 88.9 109.22))
-    (stroke (width 0) (type default) (color 0 0 0 0))
-  )
-  (wire (pts (xy 31.75 64.77) (xy 31.75 83.82))
-    (stroke (width 0) (type default) (color 0 0 0 0))
-  )
-  (wire (pts (xy 45.72 130.81) (xy 45.72 137.16))
-    (stroke (width 0) (type default) (color 0 0 0 0))
-  )
-  (wire (pts (xy 45.72 64.77) (xy 31.75 64.77))
-    (stroke (width 0) (type default) (color 0 0 0 0))
-  )
-  (wire (pts (xy 133.35 81.28) (xy 140.97 81.28))
-    (stroke (width 0) (type default) (color 0 0 0 0))
-  )
-  (wire (pts (xy 31.75 101.6) (xy 45.72 101.6))
-    (stroke (width 0) (type default) (color 0 0 0 0))
-  )
-  (wire (pts (xy 78.74 105.41) (xy 88.9 105.41))
-    (stroke (width 0) (type default) (color 0 0 0 0))
-  )
-  (wire (pts (xy 31.75 83.82) (xy 31.75 101.6))
-    (stroke (width 0) (type default) (color 0 0 0 0))
-  )
   (wire (pts (xy 31.75 101.6) (xy 31.75 110.49))
     (stroke (width 0) (type default) (color 0 0 0 0))
@@
     (effects (font (size 1.27 1.27)) (justify left bottom))
   )
-  (label "VOLUME" (at 78.74 113.03 0)
-    (effects (font (size 1.27 1.27)) (justify left bottom))
-  )
   (label "BCLK" (at 140.97 120.65 0)
     (effects (font (size 1.27 1.27)) (justify left bottom))
   )
-  (label "VIBRATO" (at 78.74 109.22 0)
-    (effects (font (size 1.27 1.27)) (justify left bottom))
-  )
   (label "SCL" (at 81.28 69.85 0)
     (effects (font (size 1.27 1.27)) (justify left bottom))
@@
     (effects (font (size 1.27 1.27)) (justify left bottom))
   )
+  (label "SENSITIVITY" (at 78.74 62.23 0)
+    (effects (font (size 1.27 1.27)) (justify left bottom))
+  )
   (label "3V3" (at 62.23 110.49 0)
     (effects (font (size 1.27 1.27)) (justify left bottom))
@@
     (effects (font (size 1.27 1.27)) (justify left bottom))
   )
+  (label "VOLUME" (at 78.74 77.47 0)
+    (effects (font (size 1.27 1.27)) (justify left bottom))
+  )
   (label "GND2" (at 88.9 144.78 0)
     (effects (font (size 1.27 1.27)) (justify left bottom))
@@
     (effects (font (size 1.27 1.27)) (justify left bottom))
   )
-  (label "SENSITIVITY" (at 78.74 105.41 0)
-    (effects (font (size 1.27 1.27)) (justify left bottom))
-  )
   (label "GND1" (at 78.74 93.98 0)
     (effects (font (size 1.27 1.27)) (justify left bottom))
@@
   )
   (label "SENSITIVITY" (at 49.53 85.09 0)
+    (effects (font (size 1.27 1.27)) (justify left bottom))
+  )
+  (label "VIBRATO" (at 78.74 73.66 0)
     (effects (font (size 1.27 1.27)) (justify left bottom))
   )
@@
       (effects (font (size 1.27 1.27)) (justify right))
     )
-    (property "Footprint" "" (id 2) (at 45.72 80.01 0)
+    (property "Footprint" "Potentiometer_THT:Potentiometer_Bourns_PTA1543_Single_Slide" (id 2) (at 45.72 80.01 0)
       (effects (font (size 1.27 1.27)) hide)
     )
@@
       (effects (font (size 2.5 2.5)))
     )
-    (property "Footprint" "" (id 2) (at 91.44 52.07 0)
+    (property "Footprint" "Module:LilyGo_T7-S3" (id 2) (at 91.44 52.07 0)
       (effects (font (size 1.27 1.27)) hide)
     )
@@
       (effects (font (size 1.27 1.27)) (justify right))
     )
-    (property "Footprint" "" (id 2) (at 45.72 97.79 0)
+    (property "Footprint" "Potentiometer_THT:Potentiometer_Bourns_PTA1543_Single_Slide" (id 2) (at 45.72 97.79 0)
       (effects (font (size 1.27 1.27)) hide)
     )
@@
       (effects (font (size 1.27 1.27)) (justify left))
     )
-    (property "Footprint" "" (id 2) (at 101.6 140.97 0)
+    (property "Footprint" "Audio_Module:MAX98357A" (id 2) (at 101.6 140.97 0)
       (effects (font (size 1.27 1.27)) hide)
     )
@@
       (effects (font (size 1.27 1.27)) hide)
     )
-    (pin "")
-    (pin "")
-    (pin "")
-    (pin "")
-    (pin "")
-    (pin "")
-    (pin "")
+    (pin "1")
+    (pin "2")
+    (pin "3")
+    (pin "4")
+    (pin "5")
+    (pin "6")
+    (pin "7")
   )
   (symbol (lib_id "Device:R_Potentiometer") (at 45.72 60.96 0) (unit 1)
@@
       (effects (font (size 1.27 1.27)) (justify right))
     )
-    (property "Footprint" "" (id 2) (at 45.72 60.96 0)
+    (property "Footprint" "Potentiometer_THT:Potentiometer_Bourns_PTA1543_Single_Slide" (id 2) (at 45.72 60.96 0)
       (effects (font (size 1.27 1.27)) hide)
     )
@@
   (symbol_instances
     (path "/d61b9ed5-0bd3-47b8-89b6-669108e3ad8a"
-      (reference "RV1") (unit 1) (value "R_Potentiometer") (footprint "")
+      (reference "RV1") (unit 1) (value "R_Potentiometer") (footprint "Potentiometer_THT:Potentiometer_Bourns_PTA1543_Single_Slide")
     )
     (path "/5bf60943-95bc-46cf-ac33-c3175b4e9d86"
-      (reference "RV2") (unit 1) (value "R_Potentiometer") (footprint "")
+      (reference "RV2") (unit 1) (value "R_Potentiometer") (footprint "Potentiometer_THT:Potentiometer_Bourns_PTA1543_Single_Slide")
     )
     (path "/96e43df4-bf40-42cc-8c5e-0ba9cbd66fda"
-      (reference "RV3") (unit 1) (value "R_Potentiometer") (footprint "")
+      (reference "RV3") (unit 1) (value "R_Potentiometer") (footprint "Potentiometer_THT:Potentiometer_Bourns_PTA1543_Single_Slide")
     )
     (path "/5a11f986-ec52-4e65-9121-a1469adbd422"
@@
     )
     (path "/5c2a55d5-91a9-4454-84c3-e1edc55a5557"
-      (reference "U2") (unit 1) (value "Lilygo_T7-S3") (footprint "")
+      (reference "U2") (unit 1) (value "Lilygo_T7-S3") (footprint "Module:LilyGo_T7-S3")
     )
     (path "/d1b4ecbd-e8ea-4a68-9f99-35c8144d6436"
-      (reference "U3") (unit 1) (value "MAX98357A") (footprint "")
-    )
-  )
+      (reference "U3") (unit 1) (value "MAX98357A") (footprint "Audio_Module:MAX98357A")
+    )
+  )
